File: KiCad/projet_capteur/projet_capteur.kicad_sch (KiCad schematic)
At the start: 9 parts, among them J1 Power, J2 Digital/PWM, J3 Analog, J4 Digital/PWM

Commit message: Save sth
Parts:
- removed U5: ~, symbol Ma_lib_graphique:model_Graphite_Sensor
- U1: footprint Lib_empreint:Empreinte_OLED -> Lib_empreint:Empreinte_Bluetooth
- U2: footprint (none) -> Lib_empreint:Empreinte_Rotary_Encoder
- U3: footprint (none) -> Lib_empreint:Empreinte_OLED
Other:
- moved on the sheet: U2, U3, U4
Changed lines of the file:
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@@
 	(symbol
 		(lib_id "Ma_lib_graphique:model_Bluetooth")
-		(at 142.24 44.45 0)
+		(at 158.75 44.45 0)
 		(unit 1)
 		(exclude_from_sim no)
@@
 		(fields_autoplaced yes)
 		(property "Reference" "U2"
-			(at 153.67 31.1149 0)
-			(effects
-				(font
-					(size 1.27 1.27)
-				)
-				(justify left)
-			)
-		)
-		(property "Value" "~"
-			(at 153.67 33.02 0)
-			(effects
-				(font
-					(size 1.27 1.27)
-				)
-				(justify left)
-			)
-		)
-		(property "Footprint" ""
-			(at 142.24 44.45 0)
+			(at 170.18 31.1149 0)
+			(effects
+				(font
+					(size 1.27 1.27)
+				)
+				(justify left)
+			)
+		)
+		(property "Value" "~"
+			(at 170.18 33.02 0)
+			(effects
+				(font
+					(size 1.27 1.27)
+				)
+				(justify left)
+			)
+		)
+		(property "Footprint" "Lib_empreint:Empreinte_Rotary_Encoder"
+			(at 158.75 44.45 0)
 			(effects
 				(font
@@
 		)
 		(property "Datasheet" ""
-			(at 142.24 44.45 0)
+			(at 158.75 44.45 0)
 			(effects
 				(font
@@
 		)
 		(property "Description" ""
-			(at 142.24 44.45 0)
+			(at 158.75 44.45 0)
 			(effects
 				(font
@@
 	(symbol
 		(lib_id "Ma_lib_graphique:model_Rotary_Encoder")
-		(at 165.1 35.56 0)
+		(at 189.23 36.83 0)
 		(unit 1)
 		(exclude_from_sim no)
@@
 		(fields_autoplaced yes)
 		(property "Reference" "U3"
-			(at 173.99 26.6699 0)
-			(effects
-				(font
-					(size 1.27 1.27)
-				)
-				(justify left)
-			)
-		)
-		(property "Value" "~"
-			(at 173.99 28.575 0)
-			(effects
-				(font
-					(size 1.27 1.27)
-				)
-				(justify left)
-			)
-		)
-		(property "Footprint" ""
-			(at 165.1 35.56 0)
+			(at 198.12 27.9399 0)
+			(effects
+				(font
+					(size 1.27 1.27)
+				)
+				(justify left)
+			)
+		)
+		(property "Value" "~"
+			(at 198.12 29.845 0)
+			(effects
+				(font
+					(size 1.27 1.27)
+				)
+				(justify left)
+			)
+		)
+		(property "Footprint" "Lib_empreint:Empreinte_OLED"
+			(at 189.23 36.83 0)
 			(effects
 				(font
@@
 		)
 		(property "Datasheet" ""
-			(at 165.1 35.56 0)
+			(at 189.23 36.83 0)
 			(effects
 				(font
@@
 		)
 		(property "Description" ""
-			(at 165.1 35.56 0)
+			(at 189.23 36.83 0)
 			(effects
 				(font
@@
 	)
 	(symbol
-		(lib_id "Ma_lib_graphique:model_Graphite_Sensor")
-		(at 205.74 31.75 0)
-		(unit 1)
-		(exclude_from_sim no)
-		(in_bom yes)
-		(on_board yes)
-		(dnp no)
-		(fields_autoplaced yes)
-		(property "Reference" "U5"
-			(at 209.55 24.7649 0)
-			(effects
-				(font
-					(size 1.27 1.27)
-				)
-				(justify left)
-			)
-		)
-		(property "Value" "~"
-			(at 209.55 26.67 0)
-			(effects
-				(font
-					(size 1.27 1.27)
-				)
-				(justify left)
-			)
-		)
-		(property "Footprint" ""
-			(at 205.74 31.75 0)
+		(lib_id "Ma_lib_graphique:model_FlexSensor")
+		(at 114.3 60.96 0)
+		(unit 1)
+		(exclude_from_sim no)
+		(in_bom yes)
+		(on_board yes)
+		(dnp no)
+		(fields_autoplaced yes)
+		(property "Reference" "U4"
+			(at 121.92 54.6099 0)
+			(effects
+				(font
+					(size 1.27 1.27)
+				)
+				(justify left)
+			)
+		)
+		(property "Value" "~"
+			(at 121.92 56.515 0)
+			(effects
+				(font
+					(size 1.27 1.27)
+				)
+				(justify left)
+			)
+		)
+		(property "Footprint" "Lib_empreint:Empreinte_FlexSensor"
+			(at 114.3 60.96 0)
 			(effects
 				(font
@@
 		)
 		(property "Datasheet" ""
-			(at 205.74 31.75 0)
+			(at 114.3 60.96 0)
 			(effects
 				(font
@@
 		)
 		(property "Description" ""
-			(at 205.74 31.75 0)
-			(effects
-				(font
-					(size 1.27 1.27)
-				)
-				(hide yes)
-			)
-		)
-		(pin "1"
-		)
-		(pin "2"
-		)
-		(instances
-			(project ""
-				(path "/e63e39d7-6ac0-4ffd-8aa3-1841a4541b55"
-					(reference "U5")
-					(unit 1)
-				)
-			)
-		)
-	)
-	(symbol
-		(lib_id "Ma_lib_graphique:model_FlexSensor")
-		(at 186.69 27.94 0)
-		(unit 1)
-		(exclude_from_sim no)
-		(in_bom yes)
-		(on_board yes)
-		(dnp no)
-		(fields_autoplaced yes)
-		(property "Reference" "U4"
-			(at 194.31 21.5899 0)
-			(effects
-				(font
-					(size 1.27 1.27)
-				)
-				(justify left)
-			)
-		)
-		(property "Value" "~"
-			(at 194.31 23.495 0)
-			(effects
-				(font
-					(size 1.27 1.27)
-				)
-				(justify left)
-			)
-		)
-		(property "Footprint" "Lib_empreint:Empreinte_FlexSensor"
-			(at 186.69 27.94 0)
-			(effects
-				(font
-					(size 1.27 1.27)
-				)
-				(hide yes)
-			)
-		)
-		(property "Datasheet" ""
-			(at 186.69 27.94 0)
-			(effects
-				(font
-					(size 1.27 1.27)
-				)
-				(hide yes)
-			)
-		)
-		(property "Description" ""
-			(at 186.69 27.94 0)
+			(at 114.3 60.96 0)
 			(effects
 				(font
@@
 			)
 		)
-		(property "Footprint" "Lib_empreint:Empreinte_OLED"
+		(property "Footprint" "Lib_empreint:Empreinte_Bluetooth"
 			(at 113.03 31.75 0)
 			(effects
