File: KiCad/projet_capteur/projet_capteur.kicad_sch (KiCad schematic)
At the start: 19 parts, among them J1 Power, J2 Digital/PWM, J3 Analog, J4 Digital/PWM

Commit message: Schématique
Parts:
- added U8: ~, symbol Ma_lib_graphique:model_ConnecteurMoteur
Connections:
- net *10 is gone; now on net 10: J2.8 (Pin_8)
- net *11 is gone; now on net 11: J2.7 (Pin_7)
- net *3 is gone; now on net 3: J4.5 (Pin_5)
- net *5 is gone; now on net 5: J4.3 (Pin_3)
- net *6 is gone; now on net 6: J4.2 (Pin_2)
- net ADC is gone; now on net A0: C2.1, R6.2
- net SCL/A5 is gone; now on net A5: J2.1 (Pin_1), J3.6 (Pin_6)
- net SDA/A4 is gone; now on net A4: J2.2 (Pin_2), J3.5 (Pin_5)
- net +5V: now also U1.2 (VCC), U2.2 (VCC), U3.4 (+), U4.1 (V+), U5.1 (+), U8.2 (5V)
- net 13: now also U7.2 (SCK)
- net 2: now also U3.1 (CLK)
- net 4: now also U3.3 (SW)
- net 5V: no longer U5.1 (+)
- net A1: now also U4.2 (V-)
- net GND: now also U1.1 (GND), U2.3 (GND), U3.5 (GND), U8.1 (GND)
- net 5: now reaches U2.4 (TXD)
- net 6: now reaches U2.5 (RXD)
- net 3: now reaches U3.2 (DT)
- net 11: now reaches U7.3 (SDI/SDO)
- net 10: now reaches U7.4 (Vss)
- net A4: now reaches U1.3 (SCL)
- net A5: now reaches U1.4 (SDA)
- net *9 renamed 9
- net 9: now also U8.3 (PWM)
- no-connect marks 1 -> 15
Other:
- moved on the sheet: C1, C2, C3, C4, R1, R3, R5, R6, U5, U6
