File: KiCad/projet_capteur/projet_capteur.kicad_pcb (KiCad board)
At the start: 2 copper layers, 68.6 x 53.3 mm, 13 parts, among them J1 Power, J2 Digital/PWM, J3 Analog, J4 Digital/PWM

Commit message: Schématique
Parts:
- moved U3 56.3 mm to (161.5, 85.8), turned to 90 degrees
- moved U1 53.5 mm to (149.0, 54.8), turned to -90 degrees
- moved U2 49.6 mm to (160.0, 55.0), turned to -90 degrees
- moved U2 31.7 mm to (150.5, 89.5)
Changed lines of the file:
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@@
 	(footprint "Lib_empreint:Empreinte_Bluetooth"
 		(layer "F.Cu")
-		(at 189.25 90)
+		(at 149 54.75 -90)
 		(property "Reference" "U1"
-			(at 10 -0.5 0)
+			(at 10 -0.5 270)
 			(unlocked yes)
 			(layer "F.SilkS")
@@
 		)
 		(property "Value" "~"
-			(at 8.5 1 0)
+			(at 8.5 1 270)
 			(unlocked yes)
 			(layer "F.Fab")
@@
 		)
 		(property "Datasheet" ""
-			(at 10 0 0)
+			(at 10 0 270)
 			(unlocked yes)
 			(layer "F.Fab")
@@
 		)
 		(property "Description" ""
-			(at 10 0 0)
+			(at 10 0 270)
 			(unlocked yes)
 			(layer "F.Fab")
@@
 		)
 		(fp_text user "BLUETOOTH"
-			(at 2.5 -14.5 0)
+			(at 2.5 -14.5 270)
 			(unlocked yes)
 			(layer "F.Cu")
@@
 		)
 		(fp_text user "RXD"
-			(at 10.5 5.5 90)
+			(at 10.5 5.5 0)
 			(unlocked yes)
 			(layer "F.SilkS")
@@
 		)
 		(fp_text user "STATE"
-			(at 13 7 90)
+			(at 13 7 0)
 			(unlocked yes)
 			(layer "F.SilkS")
@@
 		)
 		(fp_text user "VCC"
-			(at 3 5.5 90)
+			(at 3 5.5 0)
 			(unlocked yes)
 			(layer "F.SilkS")
@@
 		)
 		(fp_text user "GND"
-			(at 5.5 5.5 90)
+			(at 5.5 5.5 0)
 			(unlocked yes)
 			(layer "F.SilkS")
@@
 		)
 		(fp_text user "KEY"
-			(at 0 5.5 90)
+			(at 0 5.5 0)
 			(unlocked yes)
 			(layer "F.SilkS")
@@
 		)
 		(fp_text user "TXD"
-			(at 8 5.5 90)
+			(at 8 5.5 0)
 			(unlocked yes)
 			(layer "F.SilkS")
@@
 		)
 		(pad "1" thru_hole rect
-			(at 0 0)
+			(at 0 0 270)
 			(size 2.54 2.54)
 			(drill 1)
@@
 		)
 		(pad "2" thru_hole oval
-			(at 2.5 0)
+			(at 2.5 0 270)
 			(size 2 2.54)
 			(drill 1)
@@
 		)
 		(pad "3" thru_hole oval
-			(at 5 0)
+			(at 5 0 270)
 			(size 2 2.54)
 			(drill 1)
@@
 		)
 		(pad "4" thru_hole oval
-			(at 7.5 0)
+			(at 7.5 0 270)
 			(size 2 2.54)
 			(drill 1)
@@
 		)
 		(pad "5" thru_hole oval
-			(at 10 0)
+			(at 10 0 270)
 			(size 2 2.54)
 			(drill 1)
@@
 		)
 		(pad "6" thru_hole oval
-			(at 12.5 0 180)
+			(at 12.5 0 90)
 			(size 2 2.54)
 			(drill 1)
@@
 	(footprint "Lib_empreint:Empreinte_Rotary_Encoder"
 		(layer "F.Cu")
-		(at 209.5 57.5)
+		(at 160 55 -90)
 		(property "Reference" "U2"
-			(at 0 -0.5 0)
+			(at 0 -0.5 270)
 			(unlocked yes)
 			(layer "F.SilkS")
@@
 		)
 		(property "Value" "~"
-			(at 0 1 0)
+			(at 0 1 270)
 			(unlocked yes)
 			(layer "F.Fab")
@@
 		)
 		(property "Datasheet" ""
-			(at 0 0 0)
+			(at 0 0 270)
 			(unlocked yes)
 			(layer "F.Fab")
@@
 		)
 		(property "Description" ""
-			(at 0 0 0)
+			(at 0 0 270)
 			(unlocked yes)
 			(layer "F.Fab")
@@
 		)
 		(fp_text user "Rotary Encoder"
-			(at 6.5 -14 0)
+			(at 6.5 -14 270)
 			(unlocked yes)
 			(layer "F.Cu")
@@
 		)
 		(fp_text user "+"
-			(at 9.5 4 90)
+			(at 9.5 4 0)
 			(unlocked yes)
 			(layer "F.SilkS")
@@
 		)
 		(fp_text user "SW"
-			(at 6.5 5 90)
+			(at 6.5 5 0)
 			(unlocked yes)
 			(layer "F.SilkS")
@@
 		)
 		(fp_text user "GND"
-			(at 12.5 5.5 90)
+			(at 12.5 5.5 0)
 			(unlocked yes)
 			(layer "F.SilkS")
@@
 		)
 		(fp_text user "DT"
-			(at 3.5 4.5 90)
+			(at 3.5 4.5 0)
 			(unlocked yes)
 			(layer "F.SilkS")
@@
 		)
 		(fp_text user "CLK"
-			(at 0 5.5 90)
+			(at 0 5.5 0)
 			(unlocked yes)
 			(layer "F.SilkS")
@@
 		)
 		(pad "1" thru_hole roundrect
-			(at 0 0)
+			(at 0 0 270)
 			(size 2.54 2.54)
 			(drill 1)
@@
 		)
 		(pad "2" thru_hole oval
-			(at 3 0)
+			(at 3 0 270)
 			(size 2 2.54)
 			(drill 1)
@@
 		)
 		(pad "3" thru_hole oval
-			(at 6 0)
+			(at 6 0 270)
 			(size 2 2.54)
 			(drill 1)
@@
 		)
 		(pad "4" thru_hole oval
-			(at 9 0)
+			(at 9 0 270)
 			(size 2 2.54)
 			(drill 1)
@@
 		)
 		(pad "5" thru_hole oval
-			(at 12 0)
+			(at 12 0 270)
 			(size 2 2.54)
 			(drill 1)
@@
 	(footprint "Lib_empreint:Empreinte_OLED"
 		(layer "F.Cu")
-		(at 192.85 38.95)
+		(at 161.5 85.75 90)
 		(property "Reference" "U3"
-			(at 0 17 0)
+			(at 0 17 90)
 			(layer "F.SilkS")
 			(effects
@@
 		)
 		(property "Value" "~"
-			(at 0 -2.5 0)
+			(at 0 -2.5 90)
 			(layer "F.Fab")
 			(effects
@@
 		)
 		(property "Datasheet" ""
-			(at 0 0 0)
+			(at 0 0 90)
 			(layer "F.Fab")
 			(hide yes)
@@
 		)
 		(property "Description" ""
-			(at 0 0 0)
+			(at 0 0 90)
 			(layer "F.Fab")
 			(hide yes)
@@
 		)
 		(fp_text user "VCC"
-			(at -0.5 5 90)
+			(at -0.5 5 180)
 			(unlocked yes)
 			(layer "F.SilkS")
@@
 		)
 		(fp_text user "SCL"
-			(at 2 5 90)
+			(at 2 5 180)
 			(unlocked yes)
 			(layer "F.SilkS")
@@
 		)
 		(fp_text user "GND"
-			(at -3.5 5 90)
+			(at -3.5 5 180)
 			(unlocked yes)
 			(layer "F.SilkS")
@@
 		)
 		(fp_text user "OLED"
-			(at 0 22.5 0)
+			(at 0 22.5 90)
 			(unlocked yes)
 			(layer "F.SilkS")
@@
 		)
 		(fp_text user "SDA"
-			(at 4.5 5 90)
+			(at 4.5 5 180)
 			(unlocked yes)
 			(layer "F.SilkS")
@@
 		)
 		(pad "1" thru_hole rect
-			(at -3.75 0)
+			(at -3.75 0 90)
 			(size 2 2)
 			(drill 0.8)
@@
 		)
 		(pad "2" thru_hole circle
-			(at -1.25 0)
+			(at -1.25 0 90)
 			(size 2 2)
 			(drill 0.8)
@@
 		)
 		(pad "3" thru_hole circle
-			(at 1.25 0)
+			(at 1.25 0 90)
 			(size 2 2)
 			(drill 0.8)
@@
 		)
 		(pad "4" thru_hole circle
-			(at 3.75 0)
+			(at 3.75 0 90)
 			(size 2 2)
 			(drill 0.8)
@@
 	(footprint "Lib_empreint:Empreinte_FlexSensor"
 		(layer "F.Cu")
-		(at 144 58.5)
+		(at 150.5 89.5)
 		(property "Reference" "U2"
 			(at -1 -0.5 0)
